File: Hardware/PCB/_autosave-Flight controler.kicad_sch (KiCad schematic)
At the start: 79 parts, among them J1 Screw_Terminal_01x02, J2 Conn_01x03, J3 Conn_01x03, SW1 TS-1088-AR02016, SW2 TS-1088-AR02016, U1 STM32F722RETx, U2 BQ25883RGER, U3 ICM-45686, U4 BMP580, U5 TPS63070RNMR, U6 LMR51430, X1 X322525MOB4SI, X2 Q13FC1350000400

Commit message: Add files via upload
Parts:
- added C38: 10uF, Capacitor_SMD:C_0603_1608Metric, symbol Device:C
- added C39, C40, C41, C45, C46: 100nf, Capacitor_SMD:C_0603_1608Metric, symbol Device:C
- added D2: WS2812B-2020, LED_SMD:LED_WS2812B-2020_PLCC4_2.0x2.0mm, symbol LED:WS2812B-2020
- added D3: PRTR5V0U2X, Package_TO_SOT_SMD:SOT-143, symbol Power_Protection:PRTR5V0U2X
- added J6, J7: Screw_Terminal_01x02, TerminalBlock:TerminalBlock_Xinya_XY308-2.54-2P_1x02_P2.54mm_Horizontal, symbol Connector:Screw_Terminal_01x02
- added J8: BM05B-GHS-TBT_LF__SN__N_, BM05B-GHS-TBT_LF__SN__N_:JST_BM05B-GHS-TBT_LF__SN__N_, symbol BM05B-GHS-TBT_LF__SN__N_:BM05B-GHS-TBT_LF__SN__N_
- added Q1, Q2: AO3400A, Package_TO_SOT_SMD:SOT-23, symbol Transistor_FET:AO3400A
- added R23, R26, R28, R30: 10K, Resistor_SMD:R_0201_0603Metric, symbol Device:R
- added R24, R29: 100K, Resistor_SMD:R_0201_0603Metric, symbol Device:R
- added R25, R27, R31: 100, Resistor_SMD:R_0201_0603Metric, symbol Device:R
- added S3, S4: Conn_01x03, Connector_PinHeader_2.54mm:PinHeader_1x03_P2.54mm_Vertical, symbol Connector_Generic:Conn_01x03
- renumbered J2 to S1, J3 to S2
Connections:
- net +3.3V: now also C41.1, D3.4 (VCC)
- net +5V: now also C38.2, C39.2, C40.2, D2.4 (VDD), J8.1, S3.1 (Pin_1), S4.1 (Pin_1)
- net BAT+: now also C45.2, C46.2, J6.1 (Pin_1), J7.1 (Pin_1)
- net GND: now also C38.1, C39.1, C40.1, C41.2, C45.1, C46.1, D2.2 (VSS), D3.1 (GND), J8.5, J8.S1 (SHIELD), J8.S2 (SHIELD), Q1.2 (S), Q2.2 (S), R23.2, R26.2, R28.2, R30.2, S3.3 (Pin_3), S4.3 (Pin_3)
- net SERVO3: now reaches U1.16 (PA2)
- net SERVO3: now also S3.2 (Pin_2)
- net SERVO4: now reaches U1.17 (PA3)
- net SERVO4: now also S4.2 (Pin_2)
- net STATUS_LED: now reaches U1.2 (PC13)
- net STATUS_LED: now also R31.1
- net PYRO_1: now reaches U1.33 (PB12)
- net PYRO_1: now also R25.1
- net PYRO_2: now reaches U1.34 (PB13)
- net PYRO_2: now also R27.1
- net USART6_TX: now reaches U1.37 (PC6)
- net USART6_TX: now also D3.3 (I/O2), J8.3
- net USART6_RX: now reaches U1.38 (PC7)
- net USART6_RX: now also D3.2 (I/O1), J8.2
- net PPS: now reaches U1.41 (PA8)
- net PPS: now also J8.4
- net PYRO_CON_1: now reaches U1.8 (PC0)
- net PYRO_CON_1: now also R24.2, R26.1
- net PYRO_CON_2: now reaches U1.9 (PC1)
- net PYRO_CON_2: now also R29.2, R30.1
- new net: D2.3 (DIN), R31.2
- new net: Q2.1 (G), R27.2, R28.1
- new net: J6.2 (Pin_2), Q1.3 (D), R24.1
- new net: J7.2 (Pin_2), Q2.3 (D), R29.1
- new net: Q1.1 (G), R23.1, R25.2
Other:
- note added: "GPS"
- note added: "Pyros"
- note added: "Status LED"
- moved on the sheet: S1, S2
